File: Kicad/PMOD USB UART.kicad_pcb (KiCad board)
At the start: 2 copper layers, 49.5 x 20.3 mm, 15 parts, among them J1 USB_B, J2 Pmod peripheral UART, U1 CH340C

Commit message: Small tweaks.
Other:
- board text added: "${COMMENT1}"
- board text added: "${COMPANY}"
- board text added: "${ISSUE_DATE}, ${REVISION}"
- board text removed: "2023-03-31, V1.0"
- board text removed: "https://github.com/atoomnetmarc/PMOD-USB-UART"
Changed lines of the file:
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@@
   (title_block
     (title "PMOD USB UART")
-    (date "2023-03-31")
+    (date "2023-04-01")
     (rev "V1.0")
     (company "https://github.com/atoomnetmarc/PMOD-USB-UART")
+    (comment 1 "Apache License, version 2.0")
   )
   (layers
@@
   (gr_line (start 97.79 118.11) (end 147.32 118.11)
     (stroke (width 0.1) (type default)) (layer "Edge.Cuts"))
+  (gr_text "${COMMENT1}" (at 120.65 117.475) (layer "B.SilkS")
+    (effects (font (size 1 1) (thickness 0.15)) (justify left bottom mirror))
+  )
   (gr_text "Oooo Comic Sans MS :-)" (at 114.808 108.458 345) (layer "B.SilkS")
     (effects (font (face "Comic Sans MS") (size 1.5 1.5) (thickness 0.15)) (justify mirror))
@@
     (effects (font (size 1 1) (thickness 0.15)) (justify left bottom mirror))
   )
-  (gr_text "TXD" (at 106.045 106.68) (layer "F.SilkS")
+  (gr_text "TXD" (at 104.14 106.68) (layer "F.SilkS")
+    (effects (font (size 1 1) (thickness 0.15)) (justify left))
+  )
+  (gr_text "${ISSUE_DATE}, ${REVISION}" (at 114.3 116.84) (layer "F.SilkS")
     (effects (font (size 1 1) (thickness 0.15)))
   )
-  (gr_text "2023-03-31, V1.0" (at 114.3 116.84) (layer "F.SilkS")
+  (gr_text "~{RTS}" (at 104.14 101.6) (layer "F.SilkS")
+    (effects (font (size 1 1) (thickness 0.15)) (justify left))
+  )
+  (gr_text "${COMPANY}" (at 121.92 99.06) (layer "F.SilkS")
     (effects (font (size 1 1) (thickness 0.15)))
   )
-  (gr_text "~{RTS}" (at 106.045 101.6) (layer "F.SilkS")
-    (effects (font (size 1 1) (thickness 0.15)))
-  )
-  (gr_text "https://github.com/atoomnetmarc/PMOD-USB-UART" (at 121.92 99.06) (layer "F.SilkS")
-    (effects (font (size 1 1) (thickness 0.15)))
-  )
-  (gr_text "VCC" (at 106.045 114.3) (layer "F.SilkS")
-    (effects (font (size 1 1) (thickness 0.15)))
-  )
-  (gr_text "~{CTS}" (at 106.045 109.22) (layer "F.SilkS")
-    (effects (font (size 1 1) (thickness 0.15)))
-  )
-  (gr_text "GND" (at 106.045 111.76) (layer "F.SilkS")
-    (effects (font (size 1 1) (thickness 0.15)))
-  )
-  (gr_text "RXD" (at 106.045 104.14) (layer "F.SilkS")
-    (effects (font (size 1 1) (thickness 0.15)))
+  (gr_text "VCC" (at 104.14 114.3) (layer "F.SilkS")
+    (effects (font (size 1 1) (thickness 0.15)) (justify left))
+  )
+  (gr_text "~{CTS}" (at 104.14 109.22) (layer "F.SilkS")
+    (effects (font (size 1 1) (thickness 0.15)) (justify left))
+  )
+  (gr_text "GND" (at 104.14 111.76) (layer "F.SilkS")
+    (effects (font (size 1 1) (thickness 0.15)) (justify left))
+  )
+  (gr_text "RXD" (at 104.14 104.14) (layer "F.SilkS")
+    (effects (font (size 1 1) (thickness 0.15)) (justify left))
   )
   (segment (start 133.985 112.395) (end 135.255 113.665) (width 0.44) (layer "F.Cu") (net 1))
